File: 135_sensor.kicad_sch (KiCad schematic)
At the start: 43 parts, among them J3 Conn_01x06_Female, J4 Conn_01x06_Female, U10 LM321, U11 MCP6561R, U2 LM321, U3 MCP6561R, U4 LM321, U5 MCP6561R, U6 LM321, U7 MCP6561R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

Commit message: Use through-hole connectors on bottom board
Parts:
- J3, J4: footprint Connector_PinSocket_1.27mm:PinSocket_1x06_P1.27mm_Vertical_SMD_Pin1Right -> Connector_PinSocket_1.27mm:PinSocket_1x06_P1.27mm_Vertical
Changed lines of the file:
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@@
 			)
 		)
-		(property "Footprint" "Connector_PinSocket_1.27mm:PinSocket_1x06_P1.27mm_Vertical_SMD_Pin1Right"
+		(property "Footprint" "Connector_PinSocket_1.27mm:PinSocket_1x06_P1.27mm_Vertical"
 			(at 271.78 66.04 0)
 			(effects
@@
 			)
 		)
-		(property "Footprint" "Connector_PinSocket_1.27mm:PinSocket_1x06_P1.27mm_Vertical_SMD_Pin1Right"
+		(property "Footprint" "Connector_PinSocket_1.27mm:PinSocket_1x06_P1.27mm_Vertical"
 			(at 229.87 54.61 0)
 			(effects
