File: shuttertest.kicad_pcb (KiCad board)
At the start: 2 copper layers, 52 x 104.1 mm, 74 parts, among them J1 Conn_01x20_Female, J2 Conn_01x06_Male, J3 Conn_01x06_Female, J4 Conn_01x06_Female, J5 Conn_01x06_Male, J6 Conn_01x06_Female, J7 Conn_01x06_Female, J8 AVR-ISP-6, SW1 SW_Push, U1 ATmega328PB-A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

Commit message: Add fixed series resistor to backight trimpot
Parts:
- added R17: 68, Resistor_SMD:R_0805_2012Metric_Pad1.20x1.40mm_HandSolder, B.Cu at (80.3, 59.4)
- RV2: value 100 -> 220
Connections:
- RV2 pad 2: GND -> Net-(R17-Pad1)
- RV2 pad 3: GND -> Net-(R17-Pad1)
Routing:
- net Net-(R17-Pad1): track 0.00 -> 12.4 mm
- net GND: track 169.1 -> 161.6 mm
